Commit message: Update robot.xacro

File: src/robot_description/urdf/robot.xacro (robot description, xacro)
@@ -630,5 +630,5 @@
 </joint>
 <joint name="Revolute 34" type="continuous">
-  <origin xyz="0.042768 -0.079772 0.1438" rpy="0 0 0"/>
+  <origin xyz="0.037768 -0.079772 0.1438" rpy="0 0 0"/>
   <parent link="base_link"/>
   <child link="wheel_1"/>
@@ -660,5 +660,5 @@
 </joint>
 <joint name="Revolute 42" type="continuous">
-  <origin xyz="0.242768 -0.279772 0.1438" rpy="0 0 0"/>
+  <origin xyz="0.242768 -0.284772 0.1438" rpy="0 0 0"/>
   <parent link="base_link"/>
   <child link="wheel_2"/>
@@ -666,5 +666,5 @@
 </joint>
 <joint name="Revolute 43" type="continuous">
-  <origin xyz="0.442768 -0.079772 0.1438" rpy="0 0 0"/>
+  <origin xyz="0.447768 -0.079772 0.1438" rpy="0 0 0"/>
   <parent link="base_link"/>
   <child link="wheel_3"/>
@@ -672,5 +672,5 @@
 </joint>
 <joint name="Revolute 44" type="continuous">
-  <origin xyz="0.242768 0.120228 0.1438" rpy="0 0 0"/>
+  <origin xyz="0.242768 0.125228 0.1438" rpy="0 0 0"/>
   <parent link="base_link"/>
   <child link="wheel_4"/>

Commit message: Add files via upload

File: src/robot_description/urdf/robot.xacro (robot description, xacro)
@@ -629,5 +629,5 @@
   <child link="base_link"/>
 </joint>
-<joint name="Revolute 34" type="continuous">
+<joint name="Revolute_34" type="continuous">
   <origin xyz="0.037768 -0.079772 0.1438" rpy="0 0 0"/>
   <parent link="base_link"/>
@@ -635,5 +635,5 @@
   <axis xyz="-1.0 0.0 0.0"/>
 </joint>
-<joint name="Revolute 37" type="continuous">
+<joint name="Revolute_37" type="continuous">
   <origin xyz="-0.022 0.091316 -0.033574" rpy="0 0 0"/>
   <parent link="wheel_1"/>
@@ -641,5 +641,5 @@
   <axis xyz="0.008727 0.0 0.999962"/>
 </joint>
-<joint name="Revolute 38" type="continuous">
+<joint name="Revolute_38" type="continuous">
   <origin xyz="-0.022 -0.053053 -0.081555" rpy="0 0 0"/>
   <parent link="wheel_1"/>
@@ -647,5 +647,5 @@
   <axis xyz="0.008727 0.974891 -0.222512"/>
 </joint>
-<joint name="Revolute 39" type="continuous">
+<joint name="Revolute_39" type="continuous">
   <origin xyz="-0.022 -0.09684 -0.00937" rpy="0 0 0"/>
   <parent link="wheel_1"/>
@@ -653,5 +653,5 @@
   <axis xyz="0.008727 0.433867 -0.900935"/>
 </joint>
-<joint name="Revolute 41" type="continuous">
+<joint name="Revolute_41" type="continuous">
   <origin xyz="-0.022 0.030685 -0.092326" rpy="0 0 0"/>
   <parent link="wheel_1"/>
@@ -659,5 +659,5 @@
   <axis xyz="0.008727 0.781802 0.623466"/>
 </joint>
-<joint name="Revolute 42" type="continuous">
+<joint name="Revolute_42" type="continuous">
   <origin xyz="0.242768 -0.284772 0.1438" rpy="0 0 0"/>
   <parent link="base_link"/>
@@ -665,5 +665,5 @@
   <axis xyz="-0.0 -1.0 -0.0"/>
 </joint>
-<joint name="Revolute 43" type="continuous">
+<joint name="Revolute_43" type="continuous">
   <origin xyz="0.447768 -0.079772 0.1438" rpy="0 0 0"/>
   <parent link="base_link"/>
@@ -671,5 +671,5 @@
   <axis xyz="1.0 -0.0 -0.0"/>
 </joint>
-<joint name="Revolute 44" type="continuous">
+<joint name="Revolute_44" type="continuous">
   <origin xyz="0.242768 0.125228 0.1438" rpy="0 0 0"/>
   <parent link="base_link"/>
@@ -677,5 +677,5 @@
   <axis xyz="0.0 1.0 0.0"/>
 </joint>
-<joint name="Revolute 46" type="continuous">
+<joint name="Revolute_46" type="continuous">
   <origin xyz="-0.083184 -0.022 0.050461" rpy="0 0 0"/>
   <parent link="wheel_2"/>
@@ -683,5 +683,5 @@
   <axis xyz="0.781802 0.008727 0.623466"/>
 </joint>
-<joint name="Revolute 47" type="continuous">
+<joint name="Revolute_47" type="continuous">
   <origin xyz="-0.091316 -0.022 -0.033574" rpy="0 0 0"/>
   <parent link="wheel_2"/>
@@ -689,5 +689,5 @@
   <axis xyz="-0.0 0.008727 0.999962"/>
 </joint>
-<joint name="Revolute 48" type="continuous">
+<joint name="Revolute_48" type="continuous">
   <origin xyz="-0.030685 -0.022 -0.092326" rpy="0 0 0"/>
   <parent link="wheel_2"/>
@@ -695,5 +695,5 @@
   <axis xyz="-0.781802 0.008727 0.623466"/>
 </joint>
-<joint name="Revolute 49" type="continuous">
+<joint name="Revolute_49" type="continuous">
   <origin xyz="0.053052 -0.022 -0.081555" rpy="0 0 0"/>
   <parent link="wheel_2"/>
@@ -701,5 +701,5 @@
   <axis xyz="-0.974891 0.008727 -0.222512"/>
 </joint>
-<joint name="Revolute 51" type="continuous">
+<joint name="Revolute_51" type="continuous">
   <origin xyz="0.067705 -0.022 0.06987" rpy="0 0 0"/>
   <parent link="wheel_2"/>
@@ -707,5 +707,5 @@
   <axis xyz="0.433867 0.008727 -0.900935"/>
 </joint>
-<joint name="Revolute 53" type="continuous">
+<joint name="Revolute_53" type="continuous">
   <origin xyz="0.022 -0.083184 0.050461" rpy="0 0 0"/>
   <parent link="wheel_3"/>
@@ -713,5 +713,5 @@
   <axis xyz="-0.008727 0.781802 0.623466"/>
 </joint>
-<joint name="Revolute 54" type="continuous">
+<joint name="Revolute_54" type="continuous">
   <origin xyz="0.022 -0.091316 -0.033574" rpy="0 0 0"/>
   <parent link="wheel_3"/>
@@ -719,5 +719,5 @@
   <axis xyz="-0.008727 -0.0 0.999962"/>
 </joint>
-<joint name="Revolute 55" type="continuous">
+<joint name="Revolute_55" type="continuous">
   <origin xyz="0.022 -0.030685 -0.092326" rpy="0 0 0"/>
   <parent link="wheel_3"/>
@@ -725,5 +725,5 @@
   <axis xyz="-0.008727 -0.781802 0.623466"/>
 </joint>
-<joint name="Revolute 56" type="continuous">
+<joint name="Revolute_56" type="continuous">
   <origin xyz="0.022 0.053052 -0.081555" rpy="0 0 0"/>
   <parent link="wheel_3"/>
@@ -731,5 +731,5 @@
   <axis xyz="-0.008727 -0.974891 -0.222512"/>
 </joint>
-<joint name="Revolute 57" type="continuous">
+<joint name="Revolute_57" type="continuous">
   <origin xyz="0.022 0.09684 -0.00937" rpy="0 0 0"/>
   <parent link="wheel_3"/>
@@ -737,5 +737,5 @@
   <axis xyz="-0.008727 -0.433867 -0.900935"/>
 </joint>
-<joint name="Revolute 61" type="continuous">
+<joint name="Revolute_61" type="continuous">
   <origin xyz="0.091316 0.022 -0.033574" rpy="0 0 0"/>
   <parent link="wheel_4"/>
@@ -743,5 +743,5 @@
   <axis xyz="0.0 -0.008727 0.999962"/>
 </joint>
-<joint name="Revolute 62" type="continuous">
+<joint name="Revolute_62" type="continuous">
   <origin xyz="0.030685 0.022 -0.092326" rpy="0 0 0"/>
   <parent link="wheel_4"/>
@@ -749,5 +749,5 @@
   <axis xyz="0.781802 -0.008727 0.623466"/>
 </joint>
-<joint name="Revolute 65" type="continuous">
+<joint name="Revolute_65" type="continuous">
   <origin xyz="-0.067657 0.022 0.069867" rpy="0 0 0"/>
   <parent link="wheel_4"/>
@@ -765,5 +765,5 @@
   <child link="camera_1"/>
 </joint>
-<joint name="Revolute 75" type="continuous">
+<joint name="Revolute_75" type="continuous">
   <origin xyz="0.083184 0.022 0.050461" rpy="0 0 0"/>
   <parent link="wheel_4"/>
@@ -771,5 +771,5 @@
   <axis xyz="-0.781802 -0.008727 0.623466"/>
 </joint>
-<joint name="Revolute 76" type="continuous">
+<joint name="Revolute_76" type="continuous">
   <origin xyz="-0.022 0.083184 0.050461" rpy="0 0 0"/>
   <parent link="wheel_1"/>
@@ -777,5 +777,5 @@
   <axis xyz="0.008727 -0.781802 0.623466"/>
 </joint>
-<joint name="Revolute 78" type="continuous">
+<joint name="Revolute_78" type="continuous">
   <origin xyz="-0.022 -0.067705 0.06987" rpy="0 0 0"/>
   <parent link="wheel_1"/>
@@ -783,5 +783,5 @@
   <axis xyz="0.008727 -0.433867 -0.900935"/>
 </joint>
-<joint name="Revolute 79" type="continuous">
+<joint name="Revolute_79" type="continuous">
   <origin xyz="0.09684 -0.022 -0.00937" rpy="0 0 0"/>
   <parent link="wheel_2"/>
@@ -789,5 +789,5 @@
   <axis xyz="-0.433867 0.008727 -0.900935"/>
 </joint>
-<joint name="Revolute 81" type="continuous">
+<joint name="Revolute_81" type="continuous">
   <origin xyz="0.022 0.067705 0.06987" rpy="0 0 0"/>
   <parent link="wheel_3"/>
@@ -795,5 +795,5 @@
   <axis xyz="-0.008727 0.433867 -0.900935"/>
 </joint>
-<joint name="Revolute 83" type="continuous">
+<joint name="Revolute_83" type="continuous">
   <origin xyz="-0.096807 0.022 -0.009335" rpy="0 0 0"/>
   <parent link="wheel_4"/>
@@ -801,5 +801,5 @@
   <axis xyz="0.433867 0.008727 -0.900935"/>
 </joint>
-<joint name="Revolute 84" type="continuous">
+<joint name="Revolute_84" type="continuous">
   <origin xyz="-0.053052 0.022 -0.081555" rpy="0 0 0"/>
   <parent link="wheel_4"/>
